File: ecad/ftdi_programmer_to_atmega_328p/ftdi_programmer_to_atmega_328p.sch (EAGLE design)
At the start: 5 parts

Commit message: Update FTDI Programmer to ATMEGA328p schematic & image.
Parts:
- added C3: 0.1uF/50V, PiB_capacitors:0.1UF_PTH-CER_50V-10%
Connections:
- new net N$1: C3.1, FTDI1.DTR
- new net RESET: C3.2, MCU1.PC6(D22*/PCINT14/!RESET!)
Other:
- moved on the sheet: FTDI1
Changed lines of the file:
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@@
 <part name="FTDI1" library="PiB_connectors" deviceset="FTDI" device="_PTH_VERT_MALE_2.54MM" package3d_urn="urn:adsk.eagle:package:4861768/1" value="FTDI"/>
 <part name="SUPPLY2" library="PiB_power_symbols" deviceset="GND" device=""/>
+<part name="C3" library="PiB_capacitors" deviceset="0.1UF" device="_PTH-CER_50V-10%" package3d_urn="urn:adsk.eagle:package:4945609/2" value="0.1uF/50V"/>
 </parts>
 <sheets>
@@
 <instance part="C2" gate="G$1" x="78.74" y="22.86" rot="R90"/>
 <instance part="SUPPLY6" gate="GND" x="68.58" y="22.86"/>
-<instance part="SUPPLY4" gate="5V" x="86.36" y="66.04"/>
-<instance part="FTDI1" gate="G$1" x="205.74" y="40.64"/>
-<instance part="SUPPLY2" gate="GND" x="213.36" y="27.94"/>
+<instance part="SUPPLY4" gate="5V" x="76.2" y="66.04"/>
+<instance part="FTDI1" gate="G$1" x="200.66" y="40.64"/>
+<instance part="SUPPLY2" gate="GND" x="208.28" y="27.94"/>
+<instance part="C3" gate="G$1" x="215.9" y="43.18" rot="R90"/>
 </instances>
 <busses>
@@
 <segment>
 <pinref part="FTDI1" gate="G$1" pin="GND"/>
-<wire x1="213.36" y1="33.02" x2="210.82" y2="33.02" width="0.1524" layer="91"/>
-<wire x1="213.36" y1="30.48" x2="213.36" y2="33.02" width="0.1524" layer="91"/>
+<wire x1="208.28" y1="33.02" x2="205.74" y2="33.02" width="0.1524" layer="91"/>
+<wire x1="208.28" y1="30.48" x2="208.28" y2="33.02" width="0.1524" layer="91"/>
 <pinref part="SUPPLY2" gate="GND" pin="GND"/>
 </segment>
@@
 <net name="5V" class="0">
 <segment>
-<wire x1="88.9" y1="60.96" x2="86.36" y2="60.96" width="0.1524" layer="91"/>
-<wire x1="86.36" y1="60.96" x2="86.36" y2="66.04" width="0.1524" layer="91"/>
+<wire x1="88.9" y1="60.96" x2="76.2" y2="60.96" width="0.1524" layer="91"/>
+<wire x1="76.2" y1="60.96" x2="76.2" y2="66.04" width="0.1524" layer="91"/>
 <pinref part="MCU1" gate="G$1" pin="VCC"/>
 <pinref part="MCU1" gate="G$1" pin="AVCC"/>
-<wire x1="88.9" y1="58.42" x2="86.36" y2="58.42" width="0.1524" layer="91"/>
-<wire x1="86.36" y1="58.42" x2="86.36" y2="60.96" width="0.1524" layer="91"/>
-<junction x="86.36" y="60.96"/>
+<wire x1="88.9" y1="58.42" x2="76.2" y2="58.42" width="0.1524" layer="91"/>
+<wire x1="76.2" y1="58.42" x2="76.2" y2="60.96" width="0.1524" layer="91"/>
+<junction x="76.2" y="60.96"/>
 <pinref part="SUPPLY4" gate="5V" pin="5V"/>
 </segment>
@@
 <segment>
 <pinref part="FTDI1" gate="G$1" pin="RXI"/>
-<wire x1="213.36" y1="40.64" x2="210.82" y2="40.64" width="0.1524" layer="91"/>
-<label x="213.36" y="40.64" size="1.27" layer="95" font="vector" ratio="10" xref="yes"/>
+<wire x1="208.28" y1="40.64" x2="205.74" y2="40.64" width="0.1524" layer="91"/>
+<label x="208.28" y="40.64" size="1.27" layer="95" font="vector" ratio="10" xref="yes"/>
 </segment>
 </net>
@@
 <segment>
 <pinref part="FTDI1" gate="G$1" pin="TXO"/>
-<wire x1="213.36" y1="38.1" x2="210.82" y2="38.1" width="0.1524" layer="91"/>
-<label x="213.36" y="38.1" size="1.27" layer="95" font="vector" ratio="10" xref="yes"/>
+<wire x1="208.28" y1="38.1" x2="205.74" y2="38.1" width="0.1524" layer="91"/>
+<label x="208.28" y="38.1" size="1.27" layer="95" font="vector" ratio="10" xref="yes"/>
 </segment>
 </net>
+<net name="N$1" class="0">
+<segment>
+<pinref part="FTDI1" gate="G$1" pin="DTR"/>
+<wire x1="213.36" y1="43.18" x2="205.74" y2="43.18" width="0.1524" layer="91"/>
+<pinref part="C3" gate="G$1" pin="1"/>
+</segment>
+</net>
+<net name="RESET" class="0">
+<segment>
+<pinref part="C3" gate="G$1" pin="2"/>
+<wire x1="223.52" y1="43.18" x2="220.98" y2="43.18" width="0.1524" layer="91"/>
+<label x="223.52" y="43.18" size="1.27" layer="95" font="vector" ratio="10" xref="yes"/>
+</segment>
+<segment>
+<pinref part="MCU1" gate="G$1" pin="PC6(D22*/PCINT14/!RESET!)"/>
+<wire x1="86.36" y1="63.5" x2="88.9" y2="63.5" width="0.1524" layer="91"/>
+<label x="86.36" y="63.5" size="1.27" layer="95" font="vector" ratio="10" rot="R180" xref="yes"/>
+</segment>
+</net>
